File: main/windbird_main_template.kicad_pcb (KiCad board)
At the start: 2 copper layers, 76 x 29 mm, 2 parts, among them SW1 1571300-2

Commit message: fix windbird_main_template.kicad_pcb
Parts:
- moved D1 81.9 mm to (130.0, 110.0)
- moved SW1 81.9 mm to (120.0, 108.5)
Routing:
- net /V33: track 1.59 -> 0.00 mm
- net /RST: track 1.42 -> 0.00 mm
- net /VBAT: track 1.30 -> 0.00 mm
- net GND: track 1.13 -> 0.00 mm
Changed lines of the file:
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@@
     (thickness 1.6)
     (drawings 28)
-    (tracks 8)
+    (tracks 0)
     (zones 0)
     (modules 2)
-    (nets 8)
+    (nets 5)
   )
-  (page A3)
+  (page A4)
+  (title_block
+    (title "Template for Windbird main board")
+    (date 2021-12-30)
+    (company "OpenWindMap SCIC SA")
+  )
   (layers
-    (0 F.Cu signal hide)
-    (31 B.Cu signal hide)
+    (0 F.Cu signal)
+    (31 B.Cu signal)
     (32 B.Adhes user)
     (33 F.Adhes user)
@@
     (pad_to_mask_clearance 0)
     (aux_axis_origin 0 0)
-    (grid_origin 178 125)
+    (grid_origin 100 100)
     (visible_elements FFFFFFBF)
     (pcbplotparams
@@
   )
   (net 0 "")
-  (net 1 /RST)
-  (net 2 /V33)
-  (net 3 /VBAT)
-  (net 4 GND)
-  (net 5 N-0000043)
-  (net 6 N-000005)
-  (net 7 N-000006)
+  (net 1 GND)
+  (net 2 N-0000043)
+  (net 3 N-000005)
+  (net 4 N-000006)
   (net_class Default "Ceci est la Netclass par défaut"
     (clearance 0.15)
@@
     (uvia_dia 0.508)
     (uvia_drill 0.127)
-    (add_net /RST)
-    (add_net /V33)
-    (add_net /VBAT)
     (add_net GND)
     (add_net N-0000043)
@@
   )
   (module 1571300 locked (layer F.Cu)
-    (at 198 133.5)
+    (at 120 108.5)
     (fp_text reference SW1 (at 0 3.9) (layer F.SilkS)
       (effects (font (size 1 1) (thickness 0.15)))
@@
     (pad "" smd rect (at -4.775 -1.6) (size 1.65 1.8) (layers F.Cu F.Paste F.Mask))
     (pad 1 smd rect (at -2 0.75) (size 1.5 3.5) (layers F.Cu F.Paste F.Mask)
-      (net 5 N-0000043))
+      (net 2 N-0000043))
     (pad 2 smd rect (at 2 0.75) (size 1.5 3.5) (layers F.Cu F.Paste F.Mask)
-      (net 4 GND))
+      (net 1 GND))
   )
   (module LTL1led locked (layer F.Cu)
-    (at 208 135 180)
+    (at 130 110 180)
     (fp_text reference D1 (at 0 -2 180) (layer F.SilkS)
       (effects (font (size 1 1) (thickness 0.15)))
@@
     )
     (pad 2 thru_hole circle (at 0 0 180) (size 1.5 1.5) (drill 0.7071) (layers *.Cu *.Mask F.SilkS)
-      (net 4 GND))
+      (net 1 GND))
     (pad 1 thru_hole rect (at 2.54 -0.01524 180) (size 1.5 1.5) (drill 0.7071) (layers *.Cu *.Mask F.SilkS)
-      (net 7 N-000006))
+      (net 4 N-000006))
     (pad 3 thru_hole circle (at -2.54 0 180) (size 1.5 1.5) (drill 0.7071) (layers *.Cu *.Mask F.SilkS)
-      (net 6 N-000005))
+      (net 3 N-000005))
   )
-  (gr_line (start 223.5 133) (end 223.5 117) (layer Cmts.User) (width 0.15))
-  (gr_circle (center 248 125) (end 249.1 125) (layer Edge.Cuts) (width 0.15))
-  (gr_circle (center 178 125) (end 179.1 125) (layer Edge.Cuts) (width 0.15))
-  (gr_line (start 208 131) (end 208 144) (layer Cmts.User) (width 0.2))
-  (gr_line (start 185.96 114.143) (end 185.96 111.857) (layer Cmts.User) (width 0.15))
-  (gr_line (start 191.294 114.143) (end 185.96 114.143) (layer Cmts.User) (width 0.15))
-  (gr_line (start 191.294 111.857) (end 191.294 114.143) (layer Cmts.User) (width 0.15))
-  (gr_line (start 185.96 111.857) (end 191.294 111.857) (layer Cmts.User) (width 0.15))
-  (gr_line (start 243.69886 132.224) (end 243.69886 129.19886) (layer Cmts.User) (width 0.15))
-  (gr_line (start 246.70114 132.20114) (end 243.69886 132.224) (layer Cmts.User) (width 0.15))
-  (gr_line (start 246.70114 129.22426) (end 246.70114 132.20114) (layer Cmts.User) (width 0.15))
-  (gr_line (start 243.69886 129.19886) (end 246.70114 129.22426) (layer Cmts.User) (width 0.15))
-  (gr_line (start 239.5 133) (end 223.5 133) (layer Cmts.User) (width 0.15))
-  (gr_line (start 239.5 117) (end 239.5 133) (layer Cmts.User) (width 0.15))
-  (gr_line (start 223.5 117) (end 239.5 117) (layer Cmts.User) (width 0.15))
-  (gr_line (start 184.84968 128.35014) (end 184.84968 115.65014) (layer Cmts.User) (width 0.15))
-  (gr_line (start 210.24968 128.35014) (end 184.84968 128.35014) (layer Cmts.User) (width 0.15))
-  (gr_line (start 210.24968 115.65014) (end 210.24968 128.35014) (layer Cmts.User) (width 0.15))
-  (gr_line (start 184.84968 115.65014) (end 210.24968 115.65014) (layer Cmts.User) (width 0.15))
-  (gr_line (start 175 118) (end 175 132) (angle 90) (layer Edge.Cuts) (width 0.15))
-  (gr_line (start 182.5 110.5) (end 182.5 118) (angle 90) (layer Edge.Cuts) (width 0.15))
-  (gr_line (start 182.5 139.5) (end 182.5 132) (angle 90) (layer Edge.Cuts) (width 0.15))
-  (gr_line (start 182.5 132) (end 175 132) (angle 90) (layer Edge.Cuts) (width 0.15))
-  (gr_line (start 182.5 118) (end 175 118) (angle 90) (layer Edge.Cuts) (width 0.15))
-  (gr_line (start 198 131) (end 198 144) (angle 90) (layer Cmts.User) (width 0.2))
-  (gr_line (start 182.5 139.5) (end 251 134) (angle 90) (layer Edge.Cuts) (width 0.15))
-  (gr_line (start 251 116) (end 251 134) (angle 90) (layer Edge.Cuts) (width 0.15))
-  (gr_line (start 182.5 110.5) (end 251 116) (angle 90) (layer Edge.Cuts) (width 0.15))
-  (segment (start 190.03 122.69) (end 190.03 124.07) (width 0.15) (layer B.Cu) (net 1))
-  (segment (start 190.03 124.07) (end 190 124.1) (width 0.15) (layer B.Cu) (net 1))
-  (segment (start 187.5 121.1) (end 187.49 121.11) (width 0.3) (layer B.Cu) (net 2))
-  (segment (start 187.49 121.11) (end 187.49 122.69) (width 0.3) (layer B.Cu) (net 2))
-  (segment (start 189.25 119.1) (end 190.55 119.1) (width 0.3) (layer B.Cu) (net 3))
-  (segment (start 218.35 132.05) (end 218.5 132.2) (width 0.5) (layer B.Cu) (net 4))
-  (segment (start 218.2 131.9) (end 218.35 132.05) (width 0.5) (layer B.Cu) (net 4))
-  (segment (start 185.5 113) (end 185 113.5) (width 0.5) (layer B.Cu) (net 4))
-  (zone (net 4) (net_name GND) (layer B.Cu) (hatch edge 0.508)
+  (gr_line (start 107.96 89.143) (end 107.96 86.857) (layer Cmts.User) (width 0.15))
+  (gr_line (start 145.5 108) (end 145.5 92) (layer Cmts.User) (width 0.15))
+  (gr_circle (center 170 100) (end 171.1 100) (layer Edge.Cuts) (width 0.15))
+  (gr_circle (center 100 100) (end 101.1 100) (layer Edge.Cuts) (width 0.15))
+  (gr_line (start 130 106) (end 130 119) (layer Cmts.User) (width 0.2))
+  (gr_line (start 113.294 89.143) (end 107.96 89.143) (layer Cmts.User) (width 0.15))
+  (gr_line (start 113.294 86.857) (end 113.294 89.143) (layer Cmts.User) (width 0.15))
+  (gr_line (start 107.96 86.857) (end 113.294 86.857) (layer Cmts.User) (width 0.15))
+  (gr_line (start 165.69886 107.224) (end 165.69886 104.19886) (layer Cmts.User) (width 0.15))
+  (gr_line (start 168.70114 107.20114) (end 165.69886 107.224) (layer Cmts.User) (width 0.15))
+  (gr_line (start 168.70114 104.22426) (end 168.70114 107.20114) (layer Cmts.User) (width 0.15))
+  (gr_line (start 165.69886 104.19886) (end 168.70114 104.22426) (layer Cmts.User) (width 0.15))
+  (gr_line (start 161.5 108) (end 145.5 108) (layer Cmts.User) (width 0.15))
+  (gr_line (start 161.5 92) (end 161.5 108) (layer Cmts.User) (width 0.15))
+  (gr_line (start 145.5 92) (end 161.5 92) (layer Cmts.User) (width 0.15))
+  (gr_line (start 106.84968 103.35014) (end 106.84968 90.65014) (layer Cmts.User) (width 0.15))
+  (gr_line (start 132.24968 103.35014) (end 106.84968 103.35014) (layer Cmts.User) (width 0.15))
+  (gr_line (start 132.24968 90.65014) (end 132.24968 103.35014) (layer Cmts.User) (width 0.15))
+  (gr_line (start 106.84968 90.65014) (end 132.24968 90.65014) (layer Cmts.User) (width 0.15))
+  (gr_line (start 97 93) (end 97 107) (angle 90) (layer Edge.Cuts) (width 0.15))
+  (gr_line (start 104.5 85.5) (end 104.5 93) (angle 90) (layer Edge.Cuts) (width 0.15))
+  (gr_line (start 104.5 114.5) (end 104.5 107) (angle 90) (layer Edge.Cuts) (width 0.15))
+  (gr_line (start 104.5 107) (end 97 107) (angle 90) (layer Edge.Cuts) (width 0.15))
+  (gr_line (start 104.5 93) (end 97 93) (angle 90) (layer Edge.Cuts) (width 0.15))
+  (gr_line (start 120 106) (end 120 119) (angle 90) (layer Cmts.User) (width 0.2))
+  (gr_line (start 104.5 114.5) (end 173 109) (angle 90) (layer Edge.Cuts) (width 0.15))
+  (gr_line (start 173 91) (end 173 109) (angle 90) (layer Edge.Cuts) (width 0.15))
+  (gr_line (start 104.5 85.5) (end 173 91) (angle 90) (layer Edge.Cuts) (width 0.15))
+  (zone (net 1) (net_name GND) (layer B.Cu) (hatch edge 0.508)
     (connect_pads (clearance 0.508))
     (min_thickness 0.254)
@@
     (polygon
       (pts
-        (xy 251 134) (xy 182.5 139.5) (xy 182.5 132) (xy 175 132) (xy 175 118)
-        (xy 182.5 118) (xy 182.5 110.5) (xy 251 116)
+        (xy 173 109) (xy 104.5 114.5) (xy 104.5 107) (xy 97 107) (xy 97 93)
+        (xy 104.5 93) (xy 104.5 85.5) (xy 173 91)
       )
     )
