File: front/front.kicad_pcb (KiCad board)
At the start: 2 copper layers, 20 x 6 mm, 4 parts, among them M0 Q***

Commit message: update front board
Other:
- board text added: "P + -"
- board text added: "WB FRONT 1.0"
- board text removed: "1.1"
Changed lines of the file:
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@@
-(kicad_pcb (version 4) (host pcbnew 4.0.2-4+6225~38~ubuntu14.04.1-stable)
+(kicad_pcb (version 20171130) (host pcbnew 5.1.5+dfsg1-2build2)
   (general
-    (links 0)
-    (no_connects 0)
-    (area 98.924999 84.425 122.963096 93.41375)
     (thickness 1.6)
-    (drawings 6)
+    (drawings 7)
     (tracks 14)
     (zones 0)
@@
     (zone_45_only no)
     (trace_min 0.1)
-    (segment_width 0.2)
-    (edge_width 0.15)
     (via_size 0.62)
     (via_drill 0.25)
@@
     (uvia_min_size 0.508)
     (uvia_min_drill 0.127)
+    (edge_width 0.15)
+    (segment_width 0.2)
     (pcb_text_width 0.3)
     (pcb_text_size 1 1)
@@
     (visible_elements FFFFFF3F)
     (pcbplotparams
-      (layerselection 0x010f8_80000001)
+      (layerselection 0x010f8_ffffffff)
       (usegerberextensions false)
+      (usegerberattributes false)
+      (usegerberadvancedattributes false)
+      (creategerberjobfile false)
       (excludeedgelayer false)
       (linewidth 0.150000)
@@
       (hpglpennumber 1)
       (hpglpenspeed 20)
-      (hpglpendiameter 15)
-      (hpglpenoverlay 2)
+      (hpglpendiameter 15.000000)
       (psnegative false)
       (psa4output false)
@@
       (drillshape 0)
       (scaleselection 1)
-      (outputdirectory prod2/front/))
+      (outputdirectory "./gerber/"))
   )
   (net 0 "")
@@
     (pad 2 smd rect (at 0.762 0 90) (size 0.635 1.143) (layers F.Cu F.Paste F.Mask))
     (model smd\capacitors\C0603.wrl
-      (at (xyz 0 0 0.001))
+      (offset (xyz 0 0 0.02539999961853028))
       (scale (xyz 0.5 0.5 0.5))
       (rotate (xyz 0 0 0))
     )
   )
+  (gr_text "P + -" (at 108.9 90.25) (layer B.SilkS)
+    (effects (font (size 1.2 1.2) (thickness 0.25)) (justify mirror))
+  )
   (gr_circle (center 102 90) (end 104.1 91.8) (layer F.SilkS) (width 0.2))
-  (gr_text 1.1 (at 105.75 91.25 90) (layer F.SilkS)
-    (effects (font (size 1 1) (thickness 0.25)))
+  (gr_text "WB FRONT 1.0" (at 108.85 92) (layer B.SilkS)
+    (effects (font (size 1 1) (thickness 0.25)) (justify mirror))
   )
   (gr_line (start 119 87) (end 119 93) (angle 90) (layer Edge.Cuts) (width 0.15))
